File: master/pcb/master.kicad_pcb (KiCad board)
At the start: 2 copper layers, 54.6 x 68.6 mm, 10 parts, among them J1 CONN_01X06, J2 CONN_01X03, J3 CONN_01X20, J4 CONN_01X04, J5 CONN_01X05, J6 CONN_01X20

Commit message: master pcb layout change
Parts:
- moved R3 77.0 mm to (67.4, 97.3)
- moved D1 77.0 mm to (52.8, 106.2)
- moved J2 77.0 mm to (50.9, 79.5)
- moved J3 77.0 mm to (57.3, 61.7)
- moved J4 77.0 mm to (50.9, 69.3)
- moved J6 77.0 mm to (72.5, 61.7)
- moved R1 77.0 mm to (70.0, 111.3)
- moved J1 77.0 mm to (94.1, 110.0)
- moved J5 77.0 mm to (94.1, 92.2)
- moved R2 77.0 mm to (70.0, 108.1)
Routing:
- net Net-(J1-Pad6): track 75.3 -> 74.3 mm
- net Net-(J1-Pad5): track 77.3 -> 76.3 mm
- net Net-(J1-Pad4): track 79.6 -> 78.6 mm
- net Net-(J1-Pad3): track 82.5 -> 81.6 mm
- net Net-(J1-Pad1): track 87.1 -> 86.2 mm
- net Net-(J1-Pad2): track 84.6 -> 83.7 mm
Other:
- board size 54.6 x 68.6 mm -> 52.2 x 66 mm

Commit message: pbc modifications
Parts:
- D1: footprint LEDs:LED_D5.0mm-4 -> ledrbg:LED_D5.0mm-4; moved to B.Cu
- J1, J2, J3, J4, J5, J6, R1, R2, R3: moved to B.Cu
- moved J3 62.1 mm to (57.1, 123.8)
- moved J6 62.1 mm to (72.4, 123.8)
- moved J4 46.9 mm to (50.8, 116.2)
- moved D1 38.8 mm to (67.9, 70.5), turned to 180 degrees
- moved J1 34.4 mm to (94.0, 75.6)
- moved R1 33.8 mm to (76.8, 78.1), turned to 90 degrees
- moved J2 26.5 mm to (50.8, 106.0)
- moved R2 20.7 mm to (64.1, 88.3), turned to 90 degrees
- moved R3 11.6 mm to (67.3, 85.7), turned to 90 degrees
- moved J5 1.15 mm to (94.0, 93.3)
Routing:
- net Net-(J1-Pad1): track 86.2 -> 110.5 mm
- net Net-(J1-Pad2): track 83.7 -> 103.4 mm
- net Net-(J1-Pad3): track 81.6 -> 96.6 mm
- net Net-(D1-Pad3): track 22.3 -> 8.77 mm
- net Net-(J6-Pad15): track 21.8 -> 8.89 mm
- net Net-(J1-Pad4): track 78.6 -> 91.3 mm
- net Net-(D1-Pad1): track 18.9 -> 6.98 mm
- net Net-(J1-Pad5): track 76.3 -> 84.9 mm
- net Net-(J6-Pad14): track 23.3 -> 15.1 mm
- net Net-(J4-Pad2): track 61.1 -> 65.9 mm
- net Net-(J1-Pad6): track 74.3 -> 78.5 mm
- net Net-(D1-Pad4): track 14.7 -> 11.6 mm
- net +5V: track 76.0 -> 73.2 mm
- net Net-(J4-Pad3): track 46.6 -> 47.7 mm
- net Net-(J6-Pad16): track 6.24 -> 5.26 mm
- removed copper zone on B.Cu, net GND
Other:
- board outline removed
