File: slave/pcb/slave.kicad_pcb (KiCad board)
At the start: 2 copper layers, 24.1 x 53.3 mm, 15 parts, among them J1 CONN_01X06, J2 CONN_01X06, J3 CONN_01X02, J4 CONN_01X02, U1 ATTINY2313A-PU

Commit message: master pcb layout change
Other:
- net class c1: trace_width 0.8 -> 0.6
Changed lines of the file:
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@@
     (pad_to_mask_clearance 0.2)
     (aux_axis_origin 0 0)
-    (visible_elements FFFFFF7F)
+    (visible_elements 7FFFFFFF)
     (pcbplotparams
       (layerselection 0x00000_80000000)
@@
   (net_class c1 ""
     (clearance 0.2)
-    (trace_width 0.8)
+    (trace_width 0.6)
     (via_dia 0.6)
     (via_drill 0.4)
@@
   (segment (start 100.33 95.25) (end 102.87 92.71) (width 0.8) (layer B.Cu) (net 10))
   (segment (start 99.06 90.17) (end 104.14 90.17) (width 0.8) (layer B.Cu) (net 11))
-  (segment (start 86.36 90.17) (end 87.63 90.17) (width 0.8) (layer B.Cu) (net 12) (status 400000))
-  (segment (start 90.17 87.63) (end 91.44 87.63) (width 0.8) (layer B.Cu) (net 12) (status 800000))
+  (segment (start 86.36 90.17) (end 87.63 90.17) (width 0.8) (layer B.Cu) (net 12))
+  (segment (start 90.17 87.63) (end 91.44 87.63) (width 0.8) (layer B.Cu) (net 12))
   (segment (start 87.63 90.17) (end 90.17 87.63) (width 0.8) (layer B.Cu) (net 12))
   (segment (start 91.44 90.17) (end 90.17 90.17) (width 0.8) (layer B.Cu) (net 13))
@@
   (segment (start 87.63 102.87) (end 86.36 102.87) (width 0.8) (layer B.Cu) (net 17))
   (segment (start 90.17 105.41) (end 87.63 102.87) (width 0.8) (layer B.Cu) (net 17))
-  (segment (start 86.36 87.63) (end 87.63 87.63) (width 0.8) (layer B.Cu) (net 18) (status 400000))
-  (segment (start 90.17 77.47) (end 91.44 77.47) (width 0.8) (layer B.Cu) (net 18) (status 800000))
+  (segment (start 86.36 87.63) (end 87.63 87.63) (width 0.8) (layer B.Cu) (net 18))
+  (segment (start 90.17 77.47) (end 91.44 77.47) (width 0.8) (layer B.Cu) (net 18))
   (segment (start 88.9 78.74) (end 90.17 77.47) (width 0.8) (layer B.Cu) (net 18))
   (segment (start 88.9 86.36) (end 88.9 78.74) (width 0.8) (layer B.Cu) (net 18))
@@
   (segment (start 93.98 88.9) (end 93.98 80.01) (width 0.8) (layer B.Cu) (net 18))
   (segment (start 97.79 92.71) (end 93.98 88.9) (width 0.8) (layer B.Cu) (net 18))
-  (segment (start 91.44 73.66) (end 90.17 73.66) (width 0.8) (layer B.Cu) (net 19) (status 400000))
-  (segment (start 86.36 77.47) (end 86.36 85.09) (width 0.8) (layer B.Cu) (net 19) (status 800000))
+  (segment (start 91.44 73.66) (end 90.17 73.66) (width 0.8) (layer B.Cu) (net 19))
+  (segment (start 86.36 77.47) (end 86.36 85.09) (width 0.8) (layer B.Cu) (net 19))
   (segment (start 90.17 73.66) (end 86.36 77.47) (width 0.8) (layer B.Cu) (net 19))
   (segment (start 91.44 73.66) (end 96.52 78.74) (width 0.8) (layer B.Cu) (net 19))
+  (segment (start 97.79 87.63) (end 99.06 87.63) (width 0.8) (layer B.Cu) (net 19))
+  (segment (start 96.52 86.36) (end 97.79 87.63) (width 0.8) (layer B.Cu) (net 19))
   (segment (start 96.52 78.74) (end 96.52 86.36) (width 0.8) (layer B.Cu) (net 19))
-  (segment (start 96.52 86.36) (end 97.79 87.63) (width 0.8) (layer B.Cu) (net 19))
-  (segment (start 97.79 87.63) (end 99.06 87.63) (width 0.8) (layer B.Cu) (net 19))
   (segment (start 91.44 81.28) (end 91.44 85.09) (width 0.8) (layer B.Cu) (net 20))
   (segment (start 99.06 107.95) (end 104.14 107.95) (width 0.8) (layer B.Cu) (net 21))

Commit message: pbc modifications
Parts:
- C1: footprint Capacitors_THT:C_Disc_D3.4mm_W2.1mm_P2.50mm -> Capacitors_ThroughHole:C_Disc_D3.4mm_W2.1mm_P2.50mm; moved to B.Cu
- D1, D2, D3: moved to B.Cu
- J1: value CONN_01X06 -> row; moved to B.Cu
- J2: value CONN_01X06 -> col; moved to B.Cu
- J3: value CONN_01X02 -> i2c_conn; moved to B.Cu
- J4: value CONN_01X02 -> power_conn; moved to B.Cu
- R1, R2, R3, R4, R5, R6: footprint Resistors_THT:R_Axial_DIN0207_L6.3mm_D2.5mm_P7.62mm_Horizontal -> Resistors_ThroughHole:R_Axial_DIN0207_L6.3mm_D2.5mm_P7.62mm_Horizontal; moved to B.Cu
- U1: footprint Housings_DIP:DIP-20_W7.62mm -> Housings_DIP:DIP-20_W7.62mm_LongPads; moved to B.Cu
- moved R3 46.4 mm to (99.1, 120.0)
- moved D1 45.7 mm to (100.3, 74.9), turned to 270 degrees
- moved D2 45.7 mm to (94.0, 74.9), turned to 270 degrees
- moved D3 45.7 mm to (87.6, 74.9), turned to 270 degrees
- moved R4 39.4 mm to (99.1, 116.8)
- moved R6 35.6 mm to (94.0, 80.0)
- moved R1 32.4 mm to (99.1, 113.7)
- moved R5 28.6 mm to (97.8, 83.2)
- moved C1 24.8 mm to (101.6, 109.9), turned to 270 degrees
- moved U1 24.8 mm to (91.4, 109.9)
- moved R2 21.0 mm to (104.1, 87.0), turned to 90 degrees
- moved J3 19.7 mm to (86.4, 107.3)
- moved J4 19.7 mm to (104.1, 107.3)
- moved J2 14.6 mm to (86.4, 104.8)
- moved J1 10.8 mm to (104.1, 92.1)
Routing:
- net Net-(J3-Pad2): track 32.1 -> 30.6 mm
- net +5V: track 18.3 -> 17.0 mm
- net Net-(J3-Pad1): track 32.9 -> 31.8 mm
- net Net-(R6-Pad1): track 22.1 -> 21.5 mm
- added copper zone on F.Cu, net GND
- removed copper zone on B.Cu, net GND
Other:
- net class BIG added: clearance 0.2, trace_width 1, via_dia 1, via_drill 0.4
