File: slave/pcb/slave.sch (KiCad schematic (older format))
At the start: 15 parts, among them J1 CONN_01X06, J2 CONN_01X06, J3 CONN_01X02, J4 CONN_01X02, U1 ATTINY2313A-PU

Commit message: conn_board
Parts:
- J1, J2: footprint Pin_Headers:Pin_Header_Angled_1x06_Pitch2.54mm -> Pin_Headers:Pin_Header_Straight_1x06_Pitch2.54mm
Changed lines of the file:
@@
 F 0 "J1" H 7300 3900 50  0000 C CNN
 F 1 "CONN_01X06" V 7400 3550 50  0000 C CNN
-F 2 "Pin_Headers:Pin_Header_Angled_1x06_Pitch2.54mm" H 7300 3550 50  0001 C CNN
+F 2 "Pin_Headers:Pin_Header_Straight_1x06_Pitch2.54mm" H 7300 3550 50  0001 C CNN
 F 3 "" H 7300 3550 50  0001 C CNN
 	1    7300 3550
@@
 $EndComp
 $Comp
-L GND #PWR6
+L GND #PWR01
 U 1 1 59779B70
 P 5100 5300
-F 0 "#PWR6" H 5100 5050 50  0001 C CNN
+F 0 "#PWR01" H 5100 5050 50  0001 C CNN
 F 1 "GND" H 5100 5150 50  0000 C CNN
 F 2 "" H 5100 5300 50  0001 C CNN
@@
 $EndComp
 $Comp
-L +5V #PWR5
+L +5V #PWR02
 U 1 1 59779C54
 P 5100 2800
-F 0 "#PWR5" H 5100 2650 50  0001 C CNN
+F 0 "#PWR02" H 5100 2650 50  0001 C CNN
 F 1 "+5V" H 5100 2940 50  0000 C CNN
 F 2 "" H 5100 2800 50  0001 C CNN
@@
 $EndComp
 $Comp
-L +5V #PWR8
+L +5V #PWR03
 U 1 1 59779C86
 P 8350 3450
-F 0 "#PWR8" H 8350 3300 50  0001 C CNN
+F 0 "#PWR03" H 8350 3300 50  0001 C CNN
 F 1 "+5V" H 8350 3590 50  0000 C CNN
 F 2 "" H 8350 3450 50  0001 C CNN
@@
 $EndComp
 $Comp
-L GND #PWR7
+L GND #PWR04
 U 1 1 59779DF7
 P 6700 5700
-F 0 "#PWR7" H 6700 5450 50  0001 C CNN
+F 0 "#PWR04" H 6700 5450 50  0001 C CNN
 F 1 "GND" H 6700 5550 50  0000 C CNN
 F 2 "" H 6700 5700 50  0001 C CNN
@@
 F 0 "J2" H 7350 4800 50  0000 C CNN
 F 1 "CONN_01X06" V 7450 4450 50  0000 C CNN
-F 2 "Pin_Headers:Pin_Header_Angled_1x06_Pitch2.54mm" H 7350 4450 50  0001 C CNN
+F 2 "Pin_Headers:Pin_Header_Straight_1x06_Pitch2.54mm" H 7350 4450 50  0001 C CNN
 F 3 "" H 7350 4450 50  0001 C CNN
 	1    7350 4450
@@
 Connection ~ 6700 5800
 $Comp
-L GND #PWR3
+L GND #PWR05
 U 1 1 5977A908
 P 3350 4600
-F 0 "#PWR3" H 3350 4350 50  0001 C CNN
+F 0 "#PWR05" H 3350 4350 50  0001 C CNN
 F 1 "GND" H 3350 4450 50  0000 C CNN
 F 2 "" H 3350 4600 50  0001 C CNN
@@
 $EndComp
 $Comp
-L +5V #PWR1
+L +5V #PWR06
 U 1 1 5977ACAB
 P 2150 2750
-F 0 "#PWR1" H 2150 2600 50  0001 C CNN
+F 0 "#PWR06" H 2150 2600 50  0001 C CNN
 F 1 "+5V" H 2150 2890 50  0000 C CNN
 F 2 "" H 2150 2750 50  0001 C CNN
@@
 $EndComp
 $Comp
-L GND #PWR2
+L GND #PWR07
 U 1 1 5977ACE0
 P 2150 3250
-F 0 "#PWR2" H 2150 3000 50  0001 C CNN
+F 0 "#PWR07" H 2150 3000 50  0001 C CNN
 F 1 "GND" H 2150 3100 50  0000 C CNN
 F 2 "" H 2150 3250 50  0001 C CNN
@@
 	2150 3100 2150 3250
 $Comp
-L +5V #PWR4
+L +5V #PWR08
 U 1 1 5977B114
 P 3600 2850
-F 0 "#PWR4" H 3600 2700 50  0001 C CNN
+F 0 "#PWR08" H 3600 2700 50  0001 C CNN
 F 1 "+5V" H 3600 2990 50  0000 C CNN
 F 2 "" H 3600 2850 50  0001 C CNN

Commit message: pbc modifications
Parts:
- C1: footprint Capacitors_THT:C_Disc_D3.4mm_W2.1mm_P2.50mm -> Capacitors_ThroughHole:C_Disc_D3.4mm_W2.1mm_P2.50mm
- J1: value CONN_01X06 -> row; symbol CONN_01X06 -> Conn_01x06
- J2: value CONN_01X06 -> col; symbol CONN_01X06 -> Conn_01x06
- J3: value CONN_01X02 -> i2c_conn; symbol CONN_01X02 -> Conn_01x02
- J4: value CONN_01X02 -> power_conn; symbol CONN_01X02 -> Conn_01x02
- R1, R2, R3, R4, R5, R6: footprint Resistors_THT:R_Axial_DIN0207_L6.3mm_D2.5mm_P7.62mm_Horizontal -> Resistors_ThroughHole:R_Axial_DIN0207_L6.3mm_D2.5mm_P7.62mm_Horizontal
Changed lines of the file:
@@
 EESchema Schematic File Version 2
+LIBS:slave-rescue
 LIBS:power
 LIBS:device
@@
 LIBS:contrib
 LIBS:valves
+LIBS:slave-cache
 EELAYER 25 0
 EELAYER END
@@
 $EndComp
 $Comp
-L CONN_01X06 J1
+L Conn_01x06 J1
 U 1 1 59779918
-P 7300 3550
-F 0 "J1" H 7300 3900 50  0000 C CNN
-F 1 "CONN_01X06" V 7400 3550 50  0000 C CNN
-F 2 "Pin_Headers:Pin_Header_Straight_1x06_Pitch2.54mm" H 7300 3550 50  0001 C CNN
-F 3 "" H 7300 3550 50  0001 C CNN
-	1    7300 3550
+P 7300 3500
+F 0 "J1" H 7300 3850 50  0000 C CNN
+F 1 "row" V 7400 3500 50  0000 C CNN
+F 2 "Pin_Headers:Pin_Header_Straight_1x06_Pitch2.54mm" H 7300 3500 50  0001 C CNN
+F 3 "" H 7300 3500 50  0001 C CNN
+	1    7300 3500
 	1    0    0    -1
 $EndComp
@@
 F 0 "R3" H 8180 3720 50  0000 L CNN
 F 1 "4.7k" H 8180 3660 50  0000 L CNN
-F 2 "Resistors_THT:R_Axial_DIN0207_L6.3mm_D2.5mm_P7.62mm_Horizontal" H 8150 3700 50  0001 C CNN
+F 2 "Resistors_ThroughHole:R_Axial_DIN0207_L6.3mm_D2.5mm_P7.62mm_Horizontal" H 8150 3700 50  0001 C CNN
 F 3 "" H 8150 3700 50  0001 C CNN
 	1    8150 3700
@@
 F 0 "R4" H 8530 3720 50  0000 L CNN
 F 1 "4.7k" H 8530 3660 50  0000 L CNN
-F 2 "Resistors_THT:R_Axial_DIN0207_L6.3mm_D2.5mm_P7.62mm_Horizontal" H 8500 3700 50  0001 C CNN
+F 2 "Resistors_ThroughHole:R_Axial_DIN0207_L6.3mm_D2.5mm_P7.62mm_Horizontal" H 8500 3700 50  0001 C CNN
 F 3 "" H 8500 3700 50  0001 C CNN
 	1    8500 3700
@@
 F 0 "R1" H 3630 3170 50  0000 L CNN
 F 1 "10k" H 3630 3110 50  0000 L CNN
-F 2 "Resistors_THT:R_Axial_DIN0207_L6.3mm_D2.5mm_P7.62mm_Horizontal" H 3600 3150 50  0001 C CNN
+F 2 "Resistors_ThroughHole:R_Axial_DIN0207_L6.3mm_D2.5mm_P7.62mm_Horizontal" H 3600 3150 50  0001 C CNN
 F 3 "" H 3600 3150 50  0001 C CNN
 	1    3600 3150
@@
 F 0 "R2" H 6730 5070 50  0000 L CNN
 F 1 "1k" H 6730 5010 50  0000 L CNN
-F 2 "Resistors_THT:R_Axial_DIN0207_L6.3mm_D2.5mm_P7.62mm_Horizontal" H 6700 5050 50  0001 C CNN
+F 2 "Resistors_ThroughHole:R_Axial_DIN0207_L6.3mm_D2.5mm_P7.62mm_Horizontal" H 6700 5050 50  0001 C CNN
 F 3 "" H 6700 5050 50  0001 C CNN
 	1    6700 5050
@@
 $EndComp
 $Comp
-L CONN_01X02 J3
+L Conn_01x02 J3
 U 1 1 59779AF9
-P 8950 4050
-F 0 "J3" H 8950 4200 50  0000 C CNN
-F 1 "CONN_01X02" V 9050 4050 50  0000 C CNN
-F 2 "Pin_Headers:Pin_Header_Straight_1x02_Pitch2.54mm" H 8950 4050 50  0001 C CNN
-F 3 "" H 8950 4050 50  0001 C CNN
-	1    8950 4050
+P 8950 4000
+F 0 "J3" H 8950 4150 50  0000 C CNN
+F 1 "i2c_conn" V 9050 4000 50  0000 C CNN
+F 2 "Pin_Headers:Pin_Header_Straight_1x02_Pitch2.54mm" H 8950 4000 50  0001 C CNN
+F 3 "" H 8950 4000 50  0001 C CNN
+	1    8950 4000
 	1    0    0    -1
 $EndComp
@@
 Connection ~ 8350 3500
 $Comp
-L CONN_01X06 J2
+L Conn_01x06 J2
 U 1 1 5977A334
-P 7350 4450
-F 0 "J2" H 7350 4800 50  0000 C CNN
-F 1 "CONN_01X06" V 7450 4450 50  0000 C CNN
-F 2 "Pin_Headers:Pin_Header_Straight_1x06_Pitch2.54mm" H 7350 4450 50  0001 C CNN
-F 3 "" H 7350 4450 50  0001 C CNN
-	1    7350 4450
+P 7350 4400
+F 0 "J2" H 7350 4750 50  0000 C CNN
+F 1 "col" V 7450 4400 50  0000 C CNN
+F 2 "Pin_Headers:Pin_Header_Straight_1x06_Pitch2.54mm" H 7350 4400 50  0001 C CNN
+F 3 "" H 7350 4400 50  0001 C CNN
+	1    7350 4400
 	1    0    0    -1
 $EndComp
@@
 F 0 "R5" H 3230 3970 50  0000 L CNN
 F 1 "1k" H 3230 3910 50  0000 L CNN
-F 2 "Resistors_THT:R_Axial_DIN0207_L6.3mm_D2.5mm_P7.62mm_Horizontal" H 3200 3950 50  0001 C CNN
+F 2 "Resistors_ThroughHole:R_Axial_DIN0207_L6.3mm_D2.5mm_P7.62mm_Horizontal" H 3200 3950 50  0001 C CNN
 F 3 "" H 3200 3950 50  0001 C CNN
 	1    3200 3950
@@
 F 0 "R6" H 3530 3970 50  0000 L CNN
 F 1 "1k" H 3530 3910 50  0000 L CNN
-F 2 "Resistors_THT:R_Axial_DIN0207_L6.3mm_D2.5mm_P7.62mm_Horizontal" H 3500 3950 50  0001 C CNN
+F 2 "Resistors_ThroughHole:R_Axial_DIN0207_L6.3mm_D2.5mm_P7.62mm_Horizontal" H 3500 3950 50  0001 C CNN
 F 3 "" H 3500 3950 50  0001 C CNN
 	1    3500 3950
 	1    0    0    -1
 $EndComp
-Connection ~ 6700 5450
 $Comp
 L LED D3
@@
 F 0 "C1" H 2160 3070 50  0000 L CNN
 F 1 "C_Small" H 2160 2920 50  0000 L CNN
-F 2 "Capacitors_THT:C_Disc_D3.4mm_W2.1mm_P2.50mm" H 2150 3000 50  0001 C CNN
+F 2 "Capacitors_ThroughHole:C_Disc_D3.4mm_W2.1mm_P2.50mm" H 2150 3000 50  0001 C CNN
 F 3 "" H 2150 3000 50  0001 C CNN
 	1    2150 3000
@@
 	5100 3000 5100 2800
 $Comp
-L CONN_01X02 J4
+L Conn_01x02 J4
 U 1 1 5977B868
-P 2700 3000
-F 0 "J4" H 2700 3150 50  0000 C CNN
-F 1 "CONN_01X02" V 2800 3000 50  0000 C CNN
-F 2 "Pin_Headers:Pin_Header_Straight_1x02_Pitch2.54mm" H 2700 3000 50  0001 C CNN
-F 3 "" H 2700 3000 50  0001 C CNN
-	1    2700 3000
-	1    0    0    -1
-$EndComp
+P 2700 2950
+F 0 "J4" H 2700 3100 50  0000 C CNN
+F 1 "power_conn" V 2800 2950 50  0000 C CNN
+F 2 "Pin_Headers:Pin_Header_Straight_1x02_Pitch2.54mm" H 2700 2950 50  0001 C CNN
+F 3 "" H 2700 2950 50  0001 C CNN
+	1    2700 2950
+	1    0    0    -1
+$EndComp
